Commit message: test urdf

File: src/ur16e_description/urdf/ur16e.urdf (robot description, URDF)
Before this commit: robot ur16e, 9 links, 8 joints
Links:
- removed link base_link
- removed link dummy_sensor_link
- removed link forearm_link
- removed link shoulder_link
- removed link tool0
- removed link upper_arm_link
- removed link wrist_1_link
- removed link wrist_2_link
- removed link wrist_3_link
Joints:
- removed joint elbow_joint
- removed joint sensor_mount_fixed
- removed joint shoulder_lift_joint
- removed joint shoulder_pan_joint
- removed joint wrist_1_joint
- removed joint wrist_2_joint
- removed joint wrist_3_joint
- removed joint wrist_3_link-tool0_fixed_joint
