Commit message: openrave model modified

File: src/bot_digger_description/urdf/ur16_bosch_openrave.xacro (robot description, xacro)
@@ -1,27 +1,28 @@
 <?xml version="1.0" encoding="utf-8"?>
 <robot xmlns:xacro="http://ros.org/wiki/xacro" name="or_ur">
-<xacro:macro name="robo_chisel">
+<!-- <xacro:macro name="robo_chisel"> -->
   <!-- common stuff -->
-  <!-- <xacro:include filename="$(find ur_description)/urdf/common.gazebo.xacro" /> -->
-  <!-- <xacro:property name="calibration_data" value="${load_yaml(diggerbot_calibration_file)}"/> -->
+  <xacro:include filename="$(find ur_description)/urdf/common.gazebo.xacro" />
+  <xacro:property name="diggerbot_calibration_file" value="$(find bot_digger_description)/extrinsics.yaml"/>
+  <xacro:property name="calibration_data" value="${load_yaml(diggerbot_calibration_file)}"/>
   <!-- ur10 -->
   <xacro:include filename="$(find ur16e_description)/urdf/ur16.urdf.xacro" />
   <xacro:ur16_robot prefix="chisel_"/>
   <!-- ROS base_link to UR 'Base' Coordinates transform -->
-  <!-- <link name="chisel_base"/> -->
-  <!-- <joint name="chisel_base_link-base_fixed_joint" type="fixed"> -->
+  <link name="chisel_base"/>
+  <joint name="chisel_base_link-base_fixed_joint" type="fixed">
     <!-- NOTE: this rotation is only needed as long as base_link itself is
                 not corrected wrt the real robot (ie: rotated over 180
                 degrees)
     -->
-    <!-- <origin xyz="0 0 0" rpy= "0.0 1.5707963267948966 0.0" />  -->
-    <!--"3.14 -1.5707963267948966 0.0"/-->
-    <!-- <parent link="chisel_base"/> -->
-    <!-- <child link="chisel_base_link"/> -->
-  <!-- </joint> -->
+    <origin xyz="0 0 0" rpy= "0.0 1.5707963267948966 0.0" />
+    "3.14 -1.5707963267948966 0.0"/
+    <parent link="chisel_base"/>
+    <child link="chisel_base_link"/>
+  </joint>
   <!-- end effector -->
-  <!-- <xacro:include filename="$(find bot_digger_description)/urdf/include/chisel_bosch.urdf.xacro" /> -->
+  <xacro:include filename="$(find bot_digger_description)/urdf/include/chisel_bosch.urdf.xacro" />
   <!-- attach -->
-  <!-- <xacro:ow_chisel prefix="chisel_" chassis_type="bot_digger_narrow_rack" calibration_data="${calibration_data}"/> -->
-  </xacro:macro>
+  <xacro:ow_chisel prefix="chisel_" chassis_type="bot_digger_narrow_rack" calibration_data="${calibration_data}"/>
+  <!-- </xacro:macro> -->
 </robot>

File: src/bot_digger_description/urdf/ur16_openrave.urdf (robot description, URDF)
Before this commit: robot or_ur, 9 links, 8 joints
Links:
- added link chisel_base
- added link chisel_chisel_link, mass 1.0; collision cylinder length=0.28 radius=0.015; visual cylinder length=0.28 radius=0.015
- link chisel_tool0: mass None -> 0.1
Joints:
- added joint chisel_base_link-base_fixed_joint: type fixed, parent chisel_base, child chisel_base_link, origin xyz=0 0 0 rpy=0.0 1.5707963267948966 0.0
- added joint chisel_chisel_fixed_joint: type fixed, parent chisel_tool0, child chisel_chisel_link, origin xyz=0.0 0.0 0.54 rpy=0.0 0.0 1.57

File: src/ur16e_description/urdf/ur16.urdf.xacro (robot description, xacro)
@@ -4,6 +4,6 @@
      For more information, please see http://wiki.ros.org/sw_urdf_exporter -->
 <robot xmlns:xacro="http://wiki.ros.org/xacro">
-  <!-- <xacro:include filename="$(find ur_description)/urdf/ur.transmission.xacro" /> -->
-  <!-- <xacro:include filename="$(find ur_description)/urdf/ur.gazebo.xacro" /> -->
+  <xacro:include filename="$(find ur_description)/urdf/ur.transmission.xacro" />
+  <xacro:include filename="$(find ur_description)/urdf/ur.gazebo.xacro" />
  <xacro:macro name="ur16_robot" params="prefix">
   <link
