Commit message: inverse dynamics added

File: src/bot_digger_description/urdf/ur16_openrave.urdf (robot description, URDF)
Before this commit: robot or_ur, 11 links, 10 joints
Links:
- link chisel_chisel_link: mass 1.0 -> 6.5; geometry collision cylinder length=0.1 radius=0.1; visual cylinder length=0.1 radius=0.1
Joints:
- joint chisel_chisel_fixed_joint: origin xyz=0.0 0.0 0.54 rpy=0.0 0.0 1.57 -> xyz=0.0 0.0 0.2032 rpy=0.0 0.0 1.57

Commit message: added data for testing

File: src/bot_digger_description/urdf/ur16_openrave.urdf (robot description, URDF)
Before this commit: robot or_ur, 11 links, 10 joints
Links:
- removed link chisel_dummy_sensor_link
- link chisel_chisel_link: mass 6.5 -> 12.6; geometry collision mesh filename=package://ur16e_description/meshes/base_link.STL; visual mesh filename=package://ur16e_description/meshes/base_link.STL
Joints:
- removed joint chisel_sensor_mount_fixed
- joint chisel_chisel_fixed_joint: origin xyz=0.0 0.0 0.2032 rpy=0.0 0.0 1.57 -> xyz=0.0 0.013 0.235 rpy=0.0 0.0 0

Commit message: test complete

File: src/bot_digger_description/urdf/ur16_openrave.urdf (robot description, URDF)
Before this commit: robot or_ur, 10 links, 9 joints
Links:
- added link chisel_tip_link, mass 0.1; collision box size=0.01 0.01 0.01
Joints:
- added joint chisel_tip_fixed_joint: type fixed, parent chisel_chisel_link, child chisel_tip_link, origin xyz=0 -0.013 0.576 rpy=0.0 0.0 0
